File: eagle/boards/dc_amp_1volt/dc_amp_1volt.sch (EAGLE design)
At the start: 13 parts, among them U1 LM358

Commit message: DC coupled Amp with limiter + board
Parts:
- added C1: 10u, adq_proc_components:C-POL
- added C2: 22u, adq_proc_components:C-POL
- added R10: 115, adq_proc_components:R
- added R11, R12: 5k, adq_proc_components:R
- added R4: 220, adq_proc_components:R
- added U$3: NCP1117, adq_proc_components:NCP1117
- added U$4, U$6, U$7, U$8, U$9: 1N4148, adq_proc_components:1N4148
- added U$5: BRIDGE, adq_proc_components:BRIDGE
- VDC2: value DC 6V AC 0 -> DC 5V AC 0
- VIN1: value DC 0V AC 2.5 SIN(0 0.5 1k 0 0) -> DC 0V AC 2.5 SIN(0 2.5 1k 0 0)
Connections:
- removed net DC_L: R5.1, R9.2, U1G3.P$V+, VDC2.+
- new net DC5_L: C1.+, R5.1, R9.2, U$3.VI, U1G3.P$V+, VDC2.+
- new net DC_ADJ_L: C2.+, R11.2, R4.2, U$3.VO, U$4.C
- new net N$11: R6.1, U$7.C, U$9.A
- new net N$4: R12.1, U$8.C, U$9.C
- new net N$6: R10.2, R4.1, U$3.ADJ, U$4.A
- new net N$7: R11.1, U$6.A, U$7.A
- net 0: now also C1.-, C2.-, R10.1, R12.2
- net N$1: now also U$5.1, U$5.2
- net VOUT_1: now also U$6.C, U$8.A; no longer R6.1
Other:
- note added: ".PARAM POT_A_VAL=50k POT_A_SET=0.2 POT_B_VAL=20k POT_B_SET=0.6"
- note removed: ".PARAM POT_A_VAL=50k POT_A_SET=0.25 POT_B_VAL=20k POT_B_SET=0.6"
- moved on the sheet: U1G2

Commit message: DC Amp. presets added
Parts:
- removed R8: 10k, adq_proc_components:R
- removed R9: 14k, adq_proc_components:R
- added JP1, JP2, JP3: (no value), pinhead:PINHD-1X2
- added POT_1: POT_1, adq_proc:POTENTIOMETER
- added PRESET_1, PRESET_2: PRESET-10MM, adq_proc:PRESET-10MM
- R10: value 115 -> 330
- U$1: value POT_A -> BRIDGE; device adq_proc_components:POTENTIOMETER -> adq_proc:BRIDGE; SPICEMODEL POT_A -> (none); SPICEPREFIX X -> (none)
- U$2: value POT_B -> POT_2; device adq_proc_components:POTENTIOMETER -> adq_proc:POTENTIOMETER; SPICEMODEL POT_B -> (none)
- U$5: device adq_proc_components:BRIDGE -> adq_proc:BRIDGE
Connections:
- removed net N$6: R10.2, R4.1, U$3.ADJ, U$4.A
- new net N$8: PRESET_1.A, PRESET_1.E, R10.2, R4.1, U$3.ADJ, U$4.A
- net 0: now also JP1.2, JP2.2, JP3.1, PRESET_1.S, PRESET_2.A, U$2.E; no longer R8.1, U$2.A
- net DC5_L: now also JP3.2, PRESET_2.E; no longer R9.2
- net IN_L: now also JP1.1
- net N$1: now also U$1.1, U$1.2, U$2.A; no longer U$2.E, U$5.1, U$5.2
- net N$2: now also PRESET_2.S; no longer R8.2, R9.1
- net N$3: now also POT_1.A, POT_1.S, U$5.1, U$5.2; no longer U$1.E, U$1.S
- net OUT: now also JP2.1
- net VOUT_1: now also POT_1.E; no longer U$1.A
Other:
- note added: ".PARAM POT_1_VAL=50k POT_1_SET=0.2 POT_2_VAL=20k POT_2_SET=0.6 PRESET_1_VAL=1k PRESET_1_SET=0.77 PRESET_2_VAL=20k PRESET_2_SET=0.5"
- note removed: ".PARAM POT_A_VAL=50k POT_A_SET=0.2 POT_B_VAL=20k POT_B_SET=0.6"
