File: eagle/boards/dc_amp_1volt/dc_amp_1volt.brd (EAGLE design)
At the start: 100 x 80 mm, 27 parts, among them U1 LM358

Commit message: Pre-amp board
Other:
- board size 100 x 80 mm -> 87.3 x 52.1 mm
